File: hardware/EmlaLockSafe_Controller_Board.kicad_pcb (KiCad board)
At the start: 2 copper layers, 58.4 x 62.2 mm, 16 parts, among them Q1 IRLML6244, U1 mini_esp32, U2 MicroUSBBreakout

Commit message: - Changed mounting holes to 3mm - Changed 5V & 3,3V wiring to allow to use the PCB without the RTC module
Routing:
- net +3V3: track 75.2 -> 108.3 mm
- net +5V: track 109.6 -> 90.6 mm
Other:
- board text added: "Emlalock Safe V2.1, 2021"
- board text removed: "Emlalock Safe V2.0, 2021"
